Commit message: update

File: medibotv4_description/urdf/medibotv4.xacro (robot description, xacro)
@@ -26,5 +26,5 @@
   </collision>
 </link>
-<link name="left_motor_1">
+<link name="left_motor">
   <inertial>
     <origin rpy="0 0 0" xyz="0.016444563411155556 0.06191343975327798 -0.056741856887104675"/>
@@ -35,5 +35,5 @@
     <origin rpy="0 0 0" xyz="0.0535 -0.1535 -0.2145"/>
     <geometry>
-      <mesh filename="package://medibotv4_description/meshes/left_motor_1.stl" scale="0.001 0.001 0.001"/>
+      <mesh filename="package://medibotv4_description/meshes/left_motor.stl" scale="0.001 0.001 0.001"/>
     </geometry>
     <material name="silver"/>
@@ -42,9 +42,9 @@
     <origin rpy="0 0 0" xyz="0.0535 -0.1535 -0.2145"/>
     <geometry>
-      <mesh filename="package://medibotv4_description/meshes/left_motor_1.stl" scale="0.001 0.001 0.001"/>
-    </geometry>
-  </collision>
-</link>
-<link name="right_motor_1">
+      <mesh filename="package://medibotv4_description/meshes/left_motor.stl" scale="0.001 0.001 0.001"/>
+    </geometry>
+  </collision>
+</link>
+<link name="right_motor">
   <inertial>
     <origin rpy="0 0 0" xyz="0.016260474645192965 -0.06154741876400091 -0.05676908795148311"/>
@@ -55,5 +55,5 @@
     <origin rpy="0 0 0" xyz="0.0535 0.1535 -0.2145"/>
     <geometry>
-      <mesh filename="package://medibotv4_description/meshes/right_motor_1.stl" scale="0.001 0.001 0.001"/>
+      <mesh filename="package://medibotv4_description/meshes/right_motor.stl" scale="0.001 0.001 0.001"/>
     </geometry>
     <material name="silver"/>
@@ -62,9 +62,9 @@
     <origin rpy="0 0 0" xyz="0.0535 0.1535 -0.2145"/>
     <geometry>
-      <mesh filename="package://medibotv4_description/meshes/right_motor_1.stl" scale="0.001 0.001 0.001"/>
-    </geometry>
-  </collision>
-</link>
-<link name="left_wheel_1">
+      <mesh filename="package://medibotv4_description/meshes/right_motor.stl" scale="0.001 0.001 0.001"/>
+    </geometry>
+  </collision>
+</link>
+<link name="left_wheel">
   <inertial>
     <origin rpy="0 0 0" xyz="7.953816428402094e-09 -0.030000265793469483 4.539531719971457e-08"/>
@@ -75,5 +75,5 @@
     <origin rpy="0 0 0" xyz="0.0175 -0.279 -0.16"/>
     <geometry>
-      <mesh filename="package://medibotv4_description/meshes/left_wheel_1.stl" scale="0.001 0.001 0.001"/>
+      <mesh filename="package://medibotv4_description/meshes/left_wheel.stl" scale="0.001 0.001 0.001"/>
     </geometry>
     <material name="silver"/>
@@ -82,9 +82,9 @@
     <origin rpy="0 0 0" xyz="0.0175 -0.279 -0.16"/>
     <geometry>
-      <mesh filename="package://medibotv4_description/meshes/left_wheel_1.stl" scale="0.001 0.001 0.001"/>
-    </geometry>
-  </collision>
-</link>
-<link name="right_wheel_1">
+      <mesh filename="package://medibotv4_description/meshes/left_wheel.stl" scale="0.001 0.001 0.001"/>
+    </geometry>
+  </collision>
+</link>
+<link name="right_wheel">
   <inertial>
     <origin rpy="0 0 0" xyz="7.952848390252454e-09 0.030000265792822806 -4.540530937346965e-08"/>
@@ -95,5 +95,5 @@
     <origin rpy="0 0 0" xyz="0.0175 0.279 -0.16"/>
     <geometry>
-      <mesh filename="package://medibotv4_description/meshes/right_wheel_1.stl" scale="0.001 0.001 0.001"/>
+      <mesh filename="package://medibotv4_description/meshes/right_wheel.stl" scale="0.001 0.001 0.001"/>
     </geometry>
     <material name="silver"/>
@@ -102,9 +102,9 @@
     <origin rpy="0 0 0" xyz="0.0175 0.279 -0.16"/>
     <geometry>
-      <mesh filename="package://medibotv4_description/meshes/right_wheel_1.stl" scale="0.001 0.001 0.001"/>
-    </geometry>
-  </collision>
-</link>
-<link name="bottom_panel_1">
+      <mesh filename="package://medibotv4_description/meshes/right_wheel.stl" scale="0.001 0.001 0.001"/>
+    </geometry>
+  </collision>
+</link>
+<link name="bottom_panel">
   <inertial>
     <origin rpy="0 0 0" xyz="0.023521505376344086 0.195 0.0025000000000000022"/>
@@ -115,5 +115,5 @@
     <origin rpy="0 0 0" xyz="-0.0 0.195 -0.06"/>
     <geometry>
-      <mesh filename="package://medibotv4_description/meshes/bottom_panel_1.stl" scale="0.001 0.001 0.001"/>
+      <mesh filename="package://medibotv4_description/meshes/bottom_panel.stl" scale="0.001 0.001 0.001"/>
     </geometry>
     <material name="silver"/>
@@ -122,9 +122,9 @@
     <origin rpy="0 0 0" xyz="-0.0 0.195 -0.06"/>
     <geometry>
-      <mesh filename="package://medibotv4_description/meshes/bottom_panel_1.stl" scale="0.001 0.001 0.001"/>
-    </geometry>
-  </collision>
-</link>
-<link name="circuit_panel_1">
+      <mesh filename="package://medibotv4_description/meshes/bottom_panel.stl" scale="0.001 0.001 0.001"/>
+    </geometry>
+  </collision>
+</link>
+<link name="circuit_panel">
   <inertial>
     <origin rpy="0 0 0" xyz="0.11000000000000001 0.0 0.0025000000000000022"/>
@@ -135,5 +135,5 @@
     <origin rpy="0 0 0" xyz="0.2 -0.0 -0.35"/>
     <geometry>
-      <mesh filename="package://medibotv4_description/meshes/circuit_panel_1.stl" scale="0.001 0.001 0.001"/>
+      <mesh filename="package://medibotv4_description/meshes/circuit_panel.stl" scale="0.001 0.001 0.001"/>
     </geometry>
     <material name="silver"/>
@@ -142,9 +142,9 @@
     <origin rpy="0 0 0" xyz="0.2 -0.0 -0.35"/>
     <geometry>
-      <mesh filename="package://medibotv4_description/meshes/circuit_panel_1.stl" scale="0.001 0.001 0.001"/>
-    </geometry>
-  </collision>
-</link>
-<link name="circuit_housing_1">
+      <mesh filename="package://medibotv4_description/meshes/circuit_panel.stl" scale="0.001 0.001 0.001"/>
+    </geometry>
+  </collision>
+</link>
+<link name="circuit_housing">
   <inertial>
     <origin rpy="0 0 0" xyz="0.11586679295026386 -4.768835044584394e-17 0.11525745568764251"/>
@@ -155,5 +155,5 @@
     <origin rpy="0 0 0" xyz="0.2 -0.0 -0.355"/>
     <geometry>
-      <mesh filename="package://medibotv4_description/meshes/circuit_housing_1.stl" scale="0.001 0.001 0.001"/>
+      <mesh filename="package://medibotv4_description/meshes/circuit_housing.stl" scale="0.001 0.001 0.001"/>
     </geometry>
     <material name="silver"/>
@@ -162,9 +162,9 @@
     <origin rpy="0 0 0" xyz="0.2 -0.0 -0.355"/>
     <geometry>
-      <mesh filename="package://medibotv4_description/meshes/circuit_housing_1.stl" scale="0.001 0.001 0.001"/>
-    </geometry>
-  </collision>
-</link>
-<link name="stand_1">
+      <mesh filename="package://medibotv4_description/meshes/circuit_housing.stl" scale="0.001 0.001 0.001"/>
+    </geometry>
+  </collision>
+</link>
+<link name="stand">
   <inertial>
     <origin rpy="0 0 0" xyz="-0.03 -5.005474418122885e-18 0.504332691249312"/>
@@ -175,5 +175,5 @@
     <origin rpy="0 0 0" xyz="-0.08 -0.0 -0.065"/>
     <geometry>
-      <mesh filename="package://medibotv4_description/meshes/stand_1.stl" scale="0.001 0.001 0.001"/>
+      <mesh filename="package://medibotv4_description/meshes/stand.stl" scale="0.001 0.001 0.001"/>
     </geometry>
     <material name="silver"/>
@@ -182,9 +182,9 @@
     <origin rpy="0 0 0" xyz="-0.08 -0.0 -0.065"/>
     <geometry>
-      <mesh filename="package://medibotv4_description/meshes/stand_1.stl" scale="0.001 0.001 0.001"/>
-    </geometry>
-  </collision>
-</link>
-<link name="body_1">
+      <mesh filename="package://medibotv4_description/meshes/stand.stl" scale="0.001 0.001 0.001"/>
+    </geometry>
+  </collision>
+</link>
+<link name="body">
   <inertial>
     <origin rpy="0 0 0" xyz="0.24442242538485656 1.3361487722796229e-15 0.22269634119543633"/>
@@ -195,5 +195,5 @@
     <origin rpy="0 0 0" xyz="0.2 -0.0 -0.03"/>
     <geometry>
-      <mesh filename="package://medibotv4_description/meshes/body_1.stl" scale="0.001 0.001 0.001"/>
+      <mesh filename="package://medibotv4_description/meshes/body.stl" scale="0.001 0.001 0.001"/>
     </geometry>
     <material name="silver"/>
@@ -202,9 +202,9 @@
     <origin rpy="0 0 0" xyz="0.2 -0.0 -0.03"/>
     <geometry>
-      <mesh filename="package://medibotv4_description/meshes/body_1.stl" scale="0.001 0.001 0.001"/>
-    </geometry>
-  </collision>
-</link>
-<link name="lidar_1">
+      <mesh filename="package://medibotv4_description/meshes/body.stl" scale="0.001 0.001 0.001"/>
+    </geometry>
+  </collision>
+</link>
+<link name="lidar">
   <inertial>
     <origin rpy="0 0 0" xyz="1.9660910471896997e-07 3.067430088395322e-17 0.014762029367898416"/>
@@ -215,5 +215,5 @@
     <origin rpy="0 0 0" xyz="-0.326625 -0.0 -0.225"/>
     <geometry>
-      <mesh filename="package://medibotv4_description/meshes/lidar_1.stl" scale="0.001 0.001 0.001"/>
+      <mesh filename="package://medibotv4_description/meshes/lidar.stl" scale="0.001 0.001 0.001"/>
     </geometry>
     <material name="silver"/>
@@ -222,9 +222,9 @@
     <origin rpy="0 0 0" xyz="-0.326625 -0.0 -0.225"/>
     <geometry>
-      <mesh filename="package://medibotv4_description/meshes/lidar_1.stl" scale="0.001 0.001 0.001"/>
-    </geometry>
-  </collision>
-</link>
-<link name="top_panel_1">
+      <mesh filename="package://medibotv4_description/meshes/lidar.stl" scale="0.001 0.001 0.001"/>
+    </geometry>
+  </collision>
+</link>
+<link name="top_panel">
   <inertial>
     <origin rpy="0 0 0" xyz="-0.3000421262648231 1.8731188253870525e-07 0.0156616040392335"/>
@@ -235,5 +235,5 @@
     <origin rpy="0 0 0" xyz="-0.366625 0.0 -0.47"/>
     <geometry>
-      <mesh filename="package://medibotv4_description/meshes/top_panel_1.stl" scale="0.001 0.001 0.001"/>
+      <mesh filename="package://medibotv4_description/meshes/top_panel.stl" scale="0.001 0.001 0.001"/>
     </geometry>
     <material name="silver"/>
@@ -242,9 +242,9 @@
     <origin rpy="0 0 0" xyz="-0.366625 0.0 -0.47"/>
     <geometry>
-      <mesh filename="package://medibotv4_description/meshes/top_panel_1.stl" scale="0.001 0.001 0.001"/>
-    </geometry>
-  </collision>
-</link>
-<link name="realsense_housing_1">
+      <mesh filename="package://medibotv4_description/meshes/top_panel.stl" scale="0.001 0.001 0.001"/>
+    </geometry>
+  </collision>
+</link>
+<link name="realsense_housing">
   <inertial>
     <origin rpy="0 0 0" xyz="-0.07373817098769747 7.951322418324285e-17 0.04233590361579864"/>
@@ -255,5 +255,5 @@
     <origin rpy="0 0 0" xyz="-0.171141 -0.0 -0.52"/>
     <geometry>
-      <mesh filename="package://medibotv4_description/meshes/realsense_housing_1.stl" scale="0.001 0.001 0.001"/>
+      <mesh filename="package://medibotv4_description/meshes/realsense_housing.stl" scale="0.001 0.001 0.001"/>
     </geometry>
     <material name="silver"/>
@@ -262,9 +262,9 @@
     <origin rpy="0 0 0" xyz="-0.171141 -0.0 -0.52"/>
     <geometry>
-      <mesh filename="package://medibotv4_description/meshes/realsense_housing_1.stl" scale="0.001 0.001 0.001"/>
-    </geometry>
-  </collision>
-</link>
-<link name="left_realsense_1">
+      <mesh filename="package://medibotv4_description/meshes/realsense_housing.stl" scale="0.001 0.001 0.001"/>
+    </geometry>
+  </collision>
+</link>
+<link name="left_realsense">
   <inertial>
     <origin rpy="0 0 0" xyz="0.00266926405942991 0.0011190896800006983 0.0"/>
@@ -275,5 +275,5 @@
     <origin rpy="0 0 0" xyz="-0.147314 -0.059696 -0.56"/>
     <geometry>
-      <mesh filename="package://medibotv4_description/meshes/left_realsense_1.stl" scale="0.001 0.001 0.001"/>
+      <mesh filename="package://medibotv4_description/meshes/left_realsense.stl" scale="0.001 0.001 0.001"/>
     </geometry>
     <material name="silver"/>
@@ -282,9 +282,9 @@
     <origin rpy="0 0 0" xyz="-0.147314 -0.059696 -0.56"/>
     <geometry>
-      <mesh filename="package://medibotv4_description/meshes/left_realsense_1.stl" scale="0.001 0.001 0.001"/>
-    </geometry>
-  </collision>
-</link>
-<link name="right_realsense_1">
+      <mesh filename="package://medibotv4_description/meshes/left_realsense.stl" scale="0.001 0.001 0.001"/>
+    </geometry>
+  </collision>
+</link>
+<link name="right_realsense">
   <inertial>
     <origin rpy="0 0 0" xyz="0.0026692640594299655 -0.0011190896800007816 5.551115123125783e-16"/>
@@ -295,5 +295,5 @@
     <origin rpy="0 0 0" xyz="-0.147314 0.059696 -0.56"/>
     <geometry>
-      <mesh filename="package://medibotv4_description/meshes/right_realsense_1.stl" scale="0.001 0.001 0.001"/>
+      <mesh filename="package://medibotv4_description/meshes/right_realsense.stl" scale="0.001 0.001 0.001"/>
     </geometry>
     <material name="silver"/>
@@ -302,9 +302,9 @@
     <origin rpy="0 0 0" xyz="-0.147314 0.059696 -0.56"/>
     <geometry>
-      <mesh filename="package://medibotv4_description/meshes/right_realsense_1.stl" scale="0.001 0.001 0.001"/>
-    </geometry>
-  </collision>
-</link>
-<link name="sonar_1">
+      <mesh filename="package://medibotv4_description/meshes/right_realsense.stl" scale="0.001 0.001 0.001"/>
+    </geometry>
+  </collision>
+</link>
+<link name="sonar">
   <inertial>
     <origin rpy="0 0 0" xyz="0.024761040929337313 1.4803902564637098e-17 0.03249999999999986"/>
@@ -315,5 +315,5 @@
     <origin rpy="0 0 0" xyz="-0.08 -0.0 -0.69"/>
     <geometry>
-      <mesh filename="package://medibotv4_description/meshes/sonar_1.stl" scale="0.001 0.001 0.001"/>
+      <mesh filename="package://medibotv4_description/meshes/sonar.stl" scale="0.001 0.001 0.001"/>
     </geometry>
     <material name="silver"/>
@@ -322,9 +322,9 @@
     <origin rpy="0 0 0" xyz="-0.08 -0.0 -0.69"/>
     <geometry>
-      <mesh filename="package://medibotv4_description/meshes/sonar_1.stl" scale="0.001 0.001 0.001"/>
-    </geometry>
-  </collision>
-</link>
-<link name="pan_servo_1">
+      <mesh filename="package://medibotv4_description/meshes/sonar.stl" scale="0.001 0.001 0.001"/>
+    </geometry>
+  </collision>
+</link>
+<link name="pan_servo">
   <inertial>
     <origin rpy="0 0 0" xyz="-0.0021812244512274467 -0.028563653527876792 0.05585888345427237"/>
@@ -335,5 +335,5 @@
     <origin rpy="0 0 0" xyz="-0.05 -0.0 -1.06"/>
     <geometry>
-      <mesh filename="package://medibotv4_description/meshes/pan_servo_1.stl" scale="0.001 0.001 0.001"/>
+      <mesh filename="package://medibotv4_description/meshes/pan_servo.stl" scale="0.001 0.001 0.001"/>
     </geometry>
     <material name="silver"/>
@@ -342,9 +342,9 @@
     <origin rpy="0 0 0" xyz="-0.05 -0.0 -1.06"/>
     <geometry>
-      <mesh filename="package://medibotv4_description/meshes/pan_servo_1.stl" scale="0.001 0.001 0.001"/>
-    </geometry>
-  </collision>
-</link>
-<link name="pan_tilt_mount_1">
+      <mesh filename="package://medibotv4_description/meshes/pan_servo.stl" scale="0.001 0.001 0.001"/>
+    </geometry>
+  </collision>
+</link>
+<link name="pan_tilt_mount">
   <inertial>
     <origin rpy="0 0 0" xyz="-0.001000621165341782 0.007999999999999986 0.09809881978571133"/>
@@ -355,5 +355,5 @@
     <origin rpy="0 0 0" xyz="-0.05 -0.035 -1.07"/>
     <geometry>
-      <mesh filename="package://medibotv4_description/meshes/pan_tilt_mount_1.stl" scale="0.001 0.001 0.001"/>
+      <mesh filename="package://medibotv4_description/meshes/pan_tilt_mount.stl" scale="0.001 0.001 0.001"/>
     </geometry>
     <material name="silver"/>
@@ -362,9 +362,9 @@
     <origin rpy="0 0 0" xyz="-0.05 -0.035 -1.07"/>
     <geometry>
-      <mesh filename="package://medibotv4_description/meshes/pan_tilt_mount_1.stl" scale="0.001 0.001 0.001"/>
-    </geometry>
-  </collision>
-</link>
-<link name="tilt_servo_1">
+      <mesh filename="package://medibotv4_description/meshes/pan_tilt_mount.stl" scale="0.001 0.001 0.001"/>
+    </geometry>
+  </collision>
+</link>
+<link name="tilt_servo">
   <inertial>
     <origin rpy="0 0 0" xyz="0.00024389797280190834 0.049434156703140976 -0.062402440810886306"/>
@@ -375,5 +375,5 @@
     <origin rpy="0 0 0" xyz="-0.05 -0.051 -1.27"/>
     <geometry>
-      <mesh filename="package://medibotv4_description/meshes/tilt_servo_1.stl" scale="0.001 0.001 0.001"/>
+      <mesh filename="package://medibotv4_description/meshes/tilt_servo.stl" scale="0.001 0.001 0.001"/>
     </geometry>
     <material name="silver"/>
@@ -382,9 +382,9 @@
     <origin rpy="0 0 0" xyz="-0.05 -0.051 -1.27"/>
     <geometry>
-      <mesh filename="package://medibotv4_description/meshes/tilt_servo_1.stl" scale="0.001 0.001 0.001"/>
-    </geometry>
-  </collision>
-</link>
-<link name="mount_1">
+      <mesh filename="package://medibotv4_description/meshes/tilt_servo.stl" scale="0.001 0.001 0.001"/>
+    </geometry>
+  </collision>
+</link>
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