Commit message: -

File: medibotv4_simulation/medibotv4_description/urdf/medibotv4.xacro (robot description, xacro)
@@ -563,5 +563,5 @@
   <child link="sonar"/>
 </joint>
-<joint name="pan_servo_joint" type="continuous">
+<joint name="pan_servo_joint" type="fixed">
   <origin rpy="0 0 0" xyz="-0.03 0.0 0.995"/>
   <parent link="stand"/>
@@ -579,5 +579,5 @@
   <child link="tilt_servo"/>
 </joint>
-<joint name="tilt_servo_joint" type="continuous">
+<joint name="tilt_servo_joint" type="fixed">
   <origin rpy="0 0 0" xyz="0.025 -0.016 -0.0525"/>
   <parent link="tilt_servo"/>

Commit message: working multirobot navigation

File: medibotv4_simulation/medibotv4_description/urdf/medibotv4.xacro (robot description, xacro)
@@ -563,5 +563,5 @@
   <child link="sonar"/>
 </joint>
-<joint name="pan_servo_joint" type="fixed">
+<joint name="pan_servo_joint" type="continuous">
   <origin rpy="0 0 0" xyz="-0.03 0.0 0.995"/>
   <parent link="stand"/>
@@ -579,5 +579,5 @@
   <child link="tilt_servo"/>
 </joint>
-<joint name="tilt_servo_joint" type="fixed">
+<joint name="tilt_servo_joint" type="continuous">
   <origin rpy="0 0 0" xyz="0.025 -0.016 -0.0525"/>
   <parent link="tilt_servo"/>

Commit message: edited robot color in rviz

File: medibotv4_simulation/medibotv4_description/urdf/medibotv4.xacro (robot description, xacro)
@@ -77,5 +77,5 @@
       <mesh filename="package://medibotv4_description/meshes/left_wheel.stl" scale="0.001 0.001 0.001"/>
     </geometry>
-    <material name="silver"/>
+    <material name="black"/>
   </visual>
   <collision>
@@ -97,5 +97,5 @@
       <mesh filename="package://medibotv4_description/meshes/right_wheel.stl" scale="0.001 0.001 0.001"/>
     </geometry>
-    <material name="silver"/>
+    <material name="black"/>
   </visual>
   <collision>
@@ -117,5 +117,7 @@
       <mesh filename="package://medibotv4_description/meshes/bottom_panel.stl" scale="0.001 0.001 0.001"/>
     </geometry>
-    <material name="silver"/>
+    <material name="white">
+      <color rgba="1.0 1.0 1.0 1.0"/>
+    </material>
   </visual>
   <collision>
@@ -137,5 +139,7 @@
       <mesh filename="package://medibotv4_description/meshes/circuit_panel.stl" scale="0.001 0.001 0.001"/>
     </geometry>
-    <material name="silver"/>
+    <material name="white">
+      <color rgba="1.0 1.0 1.0 1.0"/>
+    </material>
   </visual>
   <collision>
@@ -157,5 +161,7 @@
       <mesh filename="package://medibotv4_description/meshes/circuit_housing.stl" scale="0.001 0.001 0.001"/>
     </geometry>
-    <material name="silver"/>
+    <material name="white">
+      <color rgba="1.0 1.0 1.0 1.0"/>
+    </material>
   </visual>
   <collision>
@@ -197,5 +203,7 @@
       <mesh filename="package://medibotv4_description/meshes/body.stl" scale="0.001 0.001 0.001"/>
     </geometry>
-    <material name="silver"/>
+    <material name="white">
+      <color rgba="1.0 1.0 1.0 1.0"/>
+    </material>
   </visual>
   <collision>
@@ -217,5 +225,5 @@
       <mesh filename="package://medibotv4_description/meshes/lidar.stl" scale="0.001 0.001 0.001"/>
     </geometry>
-    <material name="silver"/>
+    <material name="black"/>
   </visual>
   <collision>
@@ -237,5 +245,7 @@
       <mesh filename="package://medibotv4_description/meshes/top_panel.stl" scale="0.001 0.001 0.001"/>
     </geometry>
-    <material name="silver"/>
+    <material name="white">
+      <color rgba="1.0 1.0 1.0 1.0"/>
+    </material>
   </visual>
   <collision>
@@ -257,5 +267,7 @@
       <mesh filename="package://medibotv4_description/meshes/realsense_housing.stl" scale="0.001 0.001 0.001"/>
     </geometry>
-    <material name="silver"/>
+    <material name="white">
+      <color rgba="1.0 1.0 1.0 1.0"/>
+    </material>
   </visual>
   <collision>
@@ -277,5 +289,5 @@
       <mesh filename="package://medibotv4_description/meshes/left_realsense.stl" scale="0.001 0.001 0.001"/>
     </geometry>
-    <material name="silver"/>
+    <material name="black"/>
   </visual>
   <collision>
@@ -297,5 +309,5 @@
       <mesh filename="package://medibotv4_description/meshes/right_realsense.stl" scale="0.001 0.001 0.001"/>
     </geometry>
-    <material name="silver"/>
+    <material name="black"/>
   </visual>
   <collision>
@@ -317,5 +329,7 @@
       <mesh filename="package://medibotv4_description/meshes/sonar.stl" scale="0.001 0.001 0.001"/>
     </geometry>
-    <material name="silver"/>
+    <material name="white">
+      <color rgba="1.0 1.0 1.0 1.0"/>
+    </material>
   </visual>
   <collision>
@@ -337,5 +351,7 @@
       <mesh filename="package://medibotv4_description/meshes/pan_servo.stl" scale="0.001 0.001 0.001"/>
     </geometry>
-    <material name="silver"/>
+    <material name="white">
+      <color rgba="1.0 1.0 1.0 1.0"/>
+    </material>
   </visual>
   <collision>
@@ -377,5 +393,7 @@
       <mesh filename="package://medibotv4_description/meshes/tilt_servo.stl" scale="0.001 0.001 0.001"/>
     </geometry>
-    <material name="silver"/>
+    <material name="white">
+      <color rgba="1.0 1.0 1.0 1.0"/>
+    </material>
   </visual>
   <collision>
@@ -397,5 +415,7 @@
       <mesh filename="package://medibotv4_description/meshes/mount.stl" scale="0.001 0.001 0.001"/>
     </geometry>
-    <material name="silver"/>
+    <material name="white">
+      <color rgba="1.0 1.0 1.0 1.0"/>
+    </material>
   </visual>
   <collision>
@@ -417,5 +437,5 @@
       <mesh filename="package://medibotv4_description/meshes/monitor.stl" scale="0.001 0.001 0.001"/>
     </geometry>
-    <material name="silver"/>
+    <material name="black"/>
   </visual>
   <collision>
@@ -437,5 +457,7 @@
       <mesh filename="package://medibotv4_description/meshes/camera_housing.stl" scale="0.001 0.001 0.001"/>
     </geometry>
-    <material name="silver"/>
+    <material name="white">
+      <color rgba="1.0 1.0 1.0 1.0"/>
+    </material>
   </visual>
   <collision>
@@ -457,5 +479,5 @@
       <mesh filename="package://medibotv4_description/meshes/camera.stl" scale="0.001 0.001 0.001"/>
     </geometry>
-    <material name="silver"/>
+    <material name="black"/>
   </visual>
   <collision>
@@ -477,5 +499,5 @@
       <mesh filename="package://medibotv4_description/meshes/caster.stl" scale="0.001 0.001 0.001"/>
     </geometry>
-    <material name="silver"/>
+    <material name="black"/>
   </visual>
   <collision>
